File: hardware/kicad/Athena/Clock.kicad_sch (KiCad schematic)
At the start: 7 parts, among them U1 NE556, U2 7400, U3 74LS157

Commit message: Update Athena clock schematic and verification journal
Parts:
- removed U?: 7400, symbol 74xx:7400
- added C2: 1uF, symbol Device:C_Polarized
- added C3, C4, C5: TBC, symbol Device:C
- added D1: HLT, symbol Device:LED
- added D2: ASTABLE, symbol Device:LED
- added R2: 1M, symbol Device:R
- added R3, R6: 10k, symbol Device:R
- added R4, R5, R7, R8: TBC, symbol Device:R
- added SW1: STEP (N.O.), symbol Switch:SW_Push
- added SW2: RUN / MANUAL, symbol Switch:SW_SPDT
- added SW3: HLT, symbol Switch:SW_SPST
- added unit 5 of U2
- U2: value 7400 -> SN7400
Connections:
- net +5V: now also R1.1, U1.10 (~{RST}), U1.14 (VCC), U1.14 (VCC), U1.4 (~{RST}), U3.16 (VCC), C3.1, C4.1, C5.1, R2.1, R3.1, R4.1, R5.1, R6.1, R7.1, U2.14 (VCC)
- net GND: now also C1.2, U1.7 (GND), U1.7 (GND), U3.10 (I1c), U3.11 (I0c), U3.13 (I1d), U3.14 (I0d), U3.15 (E), U3.5 (I0b), U3.6 (I1b), U3.8 (GND), C2.2, C3.2, C4.2, C5.2, D2.1 (K), SW1.1, SW2.2 (B), SW3.1 (A), U2.7 (GND)
- net at R1.2: now also RV1.1, U1.1 (DISCH)
- net CPU_CLK: now reaches U2.11
- net at U2.12: now also U2.13, U2.8
- net at U2.4: now also R5.2, SW2.3 (C)
- net ~{MODE_Q}: now reaches U2.5
- net ~{MODE_Q}: now also U2.3
- net MODE_Q: now reaches U2.6
- net MODE_Q: now also U2.2, U3.1 (S)
- net at U1.12 (THRES): now also U1.13 (DISCH), C2.1, R2.2
- net at U1.8 (TRIG): now also R3.2, SW1.2
- net MANUAL: now reaches U1.9 (OUT)
- net MANUAL: now also U3.2 (I0a)
- net at RV1.2: now also C1.1, U1.2 (THRES), U1.6 (TRIG)
- net at U2.1: now also R4.2, SW2.1 (A)
- net ASTABLE: now reaches U1.5 (OUT)
- net ASTABLE: now also U3.3 (I1a), R8.1
- net SELECTED_CLK: now reaches U3.4 (Za)
- net SELECTED_CLK: now also U2.9
- net CLOCK_ENABLE: now reaches U2.10
- net CLOCK_ENABLE: now also D1.1 (K), R6.2, SW3.2 (B)
- new net: D2.2 (A), R8.2
- new net: D1.2 (A), R7.2
- no-connect marks 0 -> 6
Other:
- note added: "1M / 1uF: nominal pulse approximately 1.1 s. Release STEP before the timing interval ends."
- note added: "Ground pin 1: MANUAL. Ground pin 4: RUN. R4/R5 values and switch physical terminal mapping: TBC."
- note added: "MANUAL"
- note added: "RUN"
- note added: "SN7400 A/B — RUN / MANUAL LATCH"
- note added: "SN7400 C/D — HLT / CPU CLOCK"
- note added: "TBC = unknown; confirm before building. U1 pins 3/11 open; RV1 unused end shown open. D2 return to GND provisional; R7/R8 unknown. C3-C5 bypass provisions: fitted parts/values TBC. U3 unused inputs shown grounded: confirm as built."
- note added: "TIMER 1 — VARIABLE-SPEED ASTABLE"
- note added: "TIMER 2 — MANUAL STEP"
- title: (none) -> Athena — complete clock circuit
- moved on the sheet: C1, R1, RV1, U1A, U1B, U2A, U2B, U2C, U2D, U3

Commit message: Update handover text and Kicad BoM and Schema
Other:
- note added: "SN7400 A/B — RUN / MANUAL LATCH / BISTABLE"
- note added: "SN74LS157N QUAD 2-to-1 MULTIPLEXER / CLOCK SELECTOR"
- note added: "TIMER 2 — MANUAL STEP / MONOSTABLE"
- note removed: "SN7400 A/B — RUN / MANUAL LATCH"
- note removed: "TIMER 2 — MANUAL STEP"
- company: (none) -> Edward Croasdell

Commit message: Add CD40106BE STEP debounce to clock schematic
Parts:
- R3: value 10k -> 47k
Connections:
- now unconnected: R3.2, SW1.2, U1.8 (TRIG)
Other:
- note added: "CD40106BE STEP DEBOUNCE R3=47k pull-up; C6=100n to GND; R9=1k in series with STEP. U4A/U4B provide two Schmitt inversions before U1 pin 8."
