File: hardware/kicad/Athena/Clock-logic.kicad_sch (KiCad schematic)
At the start: 0 parts

Commit message: Update clock logic diagram for STEP debounce
Other:
- note added: "MANUAL STEP PATH STEP → U4A/U4B CD40106B debounce U1B 556 Timer 2 → OUTPUT2 pin 9"
- note removed: "MANUAL STEP PULSE U1B — 556 Timer 2 OUTPUT2: pin 9"
Changed lines of the file:
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@@
   (title_block
     (title "Athena clock logic")
-    (date "2026-09-14")
-    (rev "1"))
+    (date "2026-09-19")
+    (rev "2"))
   (text "ATHENA — CLOCK LOGIC"
     (at 148.5 20 0)
@@
       (type none))
 )
-  (text "MANUAL STEP PULSE\nU1B — 556 Timer 2\nOUTPUT2: pin 9"
+  (text "MANUAL STEP PATH\nSTEP → U4A/U4B CD40106B debounce\nU1B 556 Timer 2 → OUTPUT2 pin 9"
     (at 51.5 91.0 0)
     (effects
@@
       (justify left))
 )
-  (embedded_fonts no))
+  (embedded_fonts no))  (text "U4 debounce: 47k pull-up / 100n to GND / 1k series STEP switch. Two Schmitt inversions preserve active-LOW trigger polarity at U1 pin 8."
+    (at 148.5 112 0)
+    (effects
+      (font
+        (size 1.27 1.27)))
+)
